File: RAM128.kicad_pcb (KiCad board)
At the start: 4 copper layers, 71.6 x 35.7 mm, 34 parts, among them J1 AppleIIBus, U1 621024, U10 74HCT32PW, U11 74AHCT1G126GW, U2 74HCT245PW, U3 74HCT273PW, U4 74HCT273PW, U5 74HCT04PW, U6 74HCT08PW, U7 74HCT32PW, U8 74HCT08PW, U9 74HCT08PW

Commit message: Good but ugly
Parts:
- removed C1, C10, C2, C5, C7, C8: 2u2, stdpads:C_0603
- removed the C3 at (122.3, 107.1)
- removed the C4 at (113.5, 107.1)
- removed the C6 at (100.7, 124.8)
- removed U5: 74HCT04PW, stdpads:TSSOP-14_4.4x5mm_P0.65mm
- added C3: 2u2, stdpads:C_0603, F.Cu at (94.4, 119.5)
- added C3: 2u2, stdpads:C_0603, F.Cu at (92.0, 119.5)
- added C3: 2u2, stdpads:C_0603, F.Cu at (116.3, 119.5)
- added C3: 2u2, stdpads:C_0603, F.Cu at (123.6, 119.5)
- added C3: 2u2, stdpads:C_0603, F.Cu at (109.0, 119.5)
- added C3: 2u2, stdpads:C_0603, F.Cu at (101.7, 119.5)
- added C4: 2u2, stdpads:C_0603, F.Cu at (105.5, 105.6)
- added C4: 2u2, stdpads:C_0603, F.Cu at (120.4, 105.6)
- added C6: 2u2, stdpads:C_0603, F.Cu at (125.0, 128.7)
- added C6: 2u2, stdpads:C_0603, F.Cu at (86.0, 127.0)
- added C6: 2u2, stdpads:C_0603, F.Cu at (75.9, 126.2)
- added C6: 2u2, stdpads:C_0603, F.Cu at (117.2, 128.7)
- added C6: 2u2, stdpads:C_0603, F.Cu at (109.6, 128.7)
- added JP1: D, Jumper:SolderJumper-2_P1.3mm_Bridged_RoundedPad1.0x1.5mm, F.Cu at (108.5, 115.8)
- added JP2: D, Jumper:SolderJumper-2_P1.3mm_Open_RoundedPad1.0x1.5mm, F.Cu at (111.8, 115.8)
- added R2: 3k3, stdpads:R_0805, F.Cu at (95.4, 116.2)
- added U12: 741G04GW, stdpads:SOT-353, F.Cu at (83.9, 127.0)
- added U13: 741G04GW, stdpads:SOT-353, F.Cu at (78.7, 127.0)
- added U14: 741G04GW, stdpads:SOT-353, F.Cu at (81.3, 127.0)
- added U15: 741G04GW, stdpads:SOT-353, F.Cu at (111.8, 128.8)
- added U16: 741G04GW, stdpads:SOT-353, F.Cu at (119.4, 128.8)
- added U17: 741G04GW, stdpads:SOT-353, F.Cu at (128.1, 113.7)
- added U19: 741G04GW, stdpads:SOT-353, F.Cu at (127.2, 128.8)
- added U20: 741G04GW, stdpads:SOT-353, F.Cu at (129.8, 128.8)
- U1: footprint stdpads:TSOP-I-32_18.4x8mm_P0.5mm -> stdpads:SOP-32_P1.27mm
- moved C9 57.3 mm to (69.2, 119.8)
- moved U2 17.5 mm to (64.9, 117.6)
- moved R1 16.8 mm to (133.6, 118.4), turned to 270 degrees
- moved FID2 12.1 mm to (64.6, 107.1)
- moved U1 11.4 mm to (80.8, 113.7), turned to 270 degrees
- moved H2 9.92 mm to (62.7, 108.8)
- moved U10 9.42 mm to (127.1, 121.8), turned to 0 degrees
- moved U4 8.14 mm to (103.2, 110.0)
- moved U6 8.09 mm to (105.2, 121.8), turned to 0 degrees
- moved FID1 7.62 mm to (62.7, 129.5)
- moved C12 7.62 mm to (63.6, 126.3)
- moved H1 7.62 mm to (65.3, 129.5)
- moved U11 7.43 mm to (122.5, 128.8)
- moved U7 6.60 mm to (97.9, 121.8), turned to 0 degrees
- moved FID3 6.35 mm to (136.9, 100.2)
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Connections:
- J1 pad 24: /DMAin -> /DMAout
- U1 pad 1: /A0 -> Net-(U1-Pad1)
- U1 pad 10: /RA16 -> /A3
- U1 pad 11: /RA15 -> /A2
- U1 pad 12: /RA14 -> /A0
- U1 pad 13: /A6 -> /RD0
- U1 pad 14: /RA12 -> /RD1
- U1 pad 15: /A5 -> /RD2
- U1 pad 16: /A4 -> GND
- U1 pad 17: /A8 -> /RD3
- U1 pad 18: /A9 -> /RD4
- U1 pad 19: /A10 -> /RD5
- U1 pad 2: /A1 -> /RA16
- U1 pad 20: /A11 -> /RD6
- U1 pad 21: /RD4 -> /RD7
- U1 pad 22: /RD5 -> /R~CS~
- U1 pad 23: /RD6 -> /A1
- U1 pad 25: /RD7 -> /A4
- U1 pad 26: /RD0 -> /A6
- U1 pad 27: /RD1 -> /A8
- U1 pad 28: /RD2 -> /A10
- U1 pad 29: /RD3 -> /R~W~
- U1 pad 3: /A2 -> /RA15
- U1 pad 30: /R~CS~ -> +5V
- U1 pad 32: GND -> +5V
- U1 pad 4: /A3 -> /RA14
- U1 pad 5: /R~W~ -> /RA12
- U1 pad 6: +5V -> /A11
- U1 pad 7: /A7 -> /A9
- U1 pad 8: +5V -> /A7
- U1 pad 9: Net-(U1-Pad9) -> /A5
- U2 pad 3: /RD2 -> /RD4
- U2 pad 4: /RD1 -> /RD5
- U2 pad 5: /RD0 -> /RD6
- U2 pad 7: /RD6 -> /RD0
- U2 pad 8: /RD5 -> /RD1
- U2 pad 9: /RD4 -> /RD2
- U4 pad 2: /RA14 -> /RA16
- U4 pad 3: /A0 -> /A3
- U4 pad 6: /RA16 -> /RA14
- U4 pad 7: /A3 -> /A0
- U6 pad 10: GND -> /A0
- U6 pad 11: /ENWR1A0 -> Net-(JP1-Pad1)
- U6 pad 12: /ENWR1 -> /INHOE
- U6 pad 13: /A0 -> /PHI0
- U6 pad 8: Net-(U6-Pad8) -> /ENWR1A0
- U6 pad 9: GND -> /ENWR1
- U7 pad 10: GND -> Net-(U19-Pad4)
- U7 pad 11: Net-(U7-Pad11) -> (no net)
- U7 pad 12: GND -> (no net)
- U7 pad 13: GND -> (no net)
- U7 pad 9: GND -> Net-(JP1-Pad2)
- U8 pad 1: Net-(U5-Pad8) -> /A12
- U8 pad 12: /A14 -> /A15
- U8 pad 13: /A15 -> /A14
- U8 pad 2: /BankAB -> /A13
- U8 pad 3: Net-(U10-Pad4) -> Net-(U10-Pad5)
- U8 pad 4: /A13 -> Net-(U15-Pad4)
- U8 pad 5: /A12 -> /BankAB
- U8 pad 6: Net-(U10-Pad5) -> Net-(U10-Pad4)
- U9 pad 4: /INHOE -> Net-(JP1-Pad1)
- U9 pad 5: /PHI0 -> /DMAin
- U9 pad 6: /RCS -> Net-(U17-Pad2)
Routing:
- net /R~CS~: track 20.6 -> 81.7 mm, vias 0 -> 2
- net /~DEVSEL~: track 67.3 -> 14.5 mm
- net /A6: track 67.0 -> 20.9 mm
- net /A4: track 63.4 -> 19.6 mm
- net /RA12: track 36.0 -> 77.2 mm, vias 2 -> 0
- net Net-(U20-Pad2): track 0.00 -> 40.8 mm, vias 0 -> 2
- net /A2: track 87.0 -> 48.0 mm, vias 3 -> 2
- net /RCS: track 38.2 -> 0.00 mm, vias 2 -> 0
- net Net-(U19-Pad4): track 0.00 -> 38.1 mm, vias 0 -> 2
- net /A7: track 71.1 -> 36.6 mm
- net /INHOE: track 9.06 -> 42.6 mm, vias 0 -> 5
- net Net-(U5-Pad8): track 31.0 -> 0.00 mm, vias 2 -> 0
- net Net-(JP1-Pad1): track 0.00 -> 30.8 mm, vias 0 -> 2
- net /A5: track 65.1 -> 34.3 mm
- net /A8: track 49.8 -> 24.4 mm
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Other:
- board size 71.6 x 35.7 mm -> 79.2 x 42 mm
- board text removed: "JLCJLCJLCJLC"

Commit message: Fabbed
Parts:
- removed the C12 at (63.6, 126.3)
- removed the C4 at (105.5, 105.6)
- removed the C4 at (120.4, 105.6)
- removed the C6 at (86.0, 127.0)
- removed the C9 at (69.2, 119.8)
- removed the H2 at (62.7, 108.8)
- removed JP1: D, Jumper:SolderJumper-2_P1.3mm_Bridged_RoundedPad1.0x1.5mm
- removed JP2: D, Jumper:SolderJumper-2_P1.3mm_Open_RoundedPad1.0x1.5mm
- added C13: 2u2, stdpads:C_0603, F.Cu at (116.2, 106.9)
- added C14: 2u2, stdpads:C_0603, F.Cu at (130.8, 106.9)
- added C15: 2u2, stdpads:C_0603, F.Cu at (131.1, 117.6)
- added C16: 10u, stdpads:C_0805, F.Cu at (73.3, 130.3)
- added C7: 2u2, stdpads:C_0603, F.Cu at (87.5, 123.0)
- added H5: , stdpads:PasteHole_1.152mm_NPTH, F.Cu at (133.1, 129.5)
- added R3: 22k, stdpads:R_0805, F.Cu at (133.2, 125.7)
- added R4: 22k, stdpads:R_0805, F.Cu at (104.8, 115.5)
- added R5: 33, stdpads:R_0805, F.Cu at (133.2, 121.5)
- added R6: 0, stdpads:R_0805, F.Cu at (104.8, 113.0)
- added R7: 0, stdpads:R_0805, F.Cu at (100.2, 113.0)
- H4: footprint stdpads:PasteHole_1.1mm_PTH -> stdpads:PasteHole_1.152mm_NPTH
- R2: value 3k3 -> 22k
- U10, U7: value 74HCT32PW -> 74AHCT32PW
- U12, U13, U14, U15, U16, U17, U19, U20: value 741G04GW -> 74AHCT1G04GW
- U6, U8, U9: value 74HCT08PW -> 74AHCT08PW
- moved H4 68.9 mm to (67.6, 108.2), turned to 270 degrees
- moved U2 18.5 mm to (83.1, 120.8)
- moved FID2 12.5 mm to (75.4, 100.7)
- moved C3 9.97 mm to (86.0, 127.5), turned to 270 degrees
- moved U1 8.98 mm to (87.2, 107.4)
- moved U4 8.15 mm to (111.3, 109.1)
- moved U3 7.80 mm to (126.0, 109.1)
- moved U17 6.55 mm to (133.2, 117.7)
- moved R1 5.11 mm to (133.2, 123.5), turned to 180 degrees
- moved FID1 5.08 mm to (67.8, 129.5)
- moved H1 5.08 mm to (70.4, 129.5)
- moved R2 4.80 mm to (100.2, 115.5), turned to 0 degrees
- moved FID3 3.68 mm to (136.9, 103.9)
- moved H3 2.90 mm to (136.9, 101.6)
- moved C4 0.90 mm to (109.6, 127.8)
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- renumbered C11 to C1, C3 to C10, C3 to C11, C3 to C12, C6 to C2, C6 to C4, C6 to C5, C3 to C8, C3 to C9, H5 to H2
Connections:
- net Net-(U13-Pad4) renamed /~A0~
- net Net-(U14-Pad4) renamed /~A1~
- net Net-(U15-Pad4) renamed /~A13~
- net Net-(U16-Pad4) renamed /~R~W
- net Net-(U17-Pad2) renamed /RCS
- net Net-(U20-Pad2) renamed /~DMAout~
- U11 pad 4: /~INH~ -> Net-(R5-Pad2)
- U2 pad 11: /D0 -> /D7
- U2 pad 12: /D1 -> /D6
- U2 pad 13: /D2 -> /D5
- U2 pad 14: /D3 -> /D4
- U2 pad 15: /D4 -> /D3
- U2 pad 16: /D5 -> /D2
- U2 pad 17: /D6 -> /D1
- U2 pad 18: /D7 -> /D0
- U2 pad 3: /RD4 -> /RD2
- U2 pad 4: /RD5 -> /RD4
- U2 pad 5: /RD6 -> /RD7
- U2 pad 6: /RD7 -> /RD0
- U2 pad 7: /RD0 -> /RD6
- U2 pad 9: /RD2 -> /RD5
- U6 pad 13: /PHI0 -> Net-(R4-Pad2)
- U7 pad 11: (no net) -> Net-(U7-Pad11)
- U7 pad 12: (no net) -> /R~W~
- U7 pad 13: (no net) -> /A13
- U9 pad 5: /DMAin -> /PHI0
Routing:
- net /RCS: track 16.8 -> 74.0 mm
- net /DMAin: track 29.3 -> 77.0 mm, vias 1 -> 2
- net +12V: track 47.5 -> 6.66 mm, vias 4 -> 1
- net Net-(R5-Pad2): track 0.00 -> 22.1 mm, vias 0 -> 2
- net /RD7: track 17.9 -> 4.08 mm
- net /PHI0: track 17.4 -> 30.3 mm
- net /RD6: track 16.2 -> 4.06 mm
- net /RD2: track 14.3 -> 26.1 mm
- net /INHOE: track 42.6 -> 54.0 mm, vias 5 -> 4
- net /A0: track 117.6 -> 128.7 mm, vias 4 -> 5
- net /RD5: track 14.5 -> 4.05 mm
- net /A1: track 91.8 -> 102.2 mm, vias 2 -> 3
- net /A3: track 79.6 -> 89.5 mm
- net /ENWR1A0: track 30.1 -> 39.8 mm
- net /ENWR1: track 28.3 -> 37.8 mm
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Other:
- board size 79.2 x 42 mm -> 74.2 x 42.7 mm
- board text added: "!"
- board text added: "Toward Rear"

Commit message: Fabbed
Parts:
- removed R6, R7: 0, stdpads:R_0805
- added SW1: DMA/ROM, stdpads:SW_DIP_SPSTx02_Slide_DSHP02TS_P1.27mm, F.Cu at (71.1, 115.1)
- R3: value 22k -> 10k
- U11: value 74AHCT1G126GW -> 74LVC1G126GW
- moved H4 3.59 mm to (70.1, 105.7)
Connections:
- net Net-(U12-Pad4) renamed /~A2~
Routing:
- net /DMAin: track 77.0 -> 123.6 mm, vias 2 -> 4
- net Net-(R4-Pad2): track 4.95 -> 48.4 mm, vias 0 -> 2
- net /RCS: track 74.0 -> 112.6 mm, vias 4 -> 6
- net Net-(R2-Pad1): track 4.95 -> 38.4 mm, vias 0 -> 2
- net /R~W~: track 88.8 -> 87.2 mm
- net GND: track 81.3 -> 80.5 mm, vias 200 -> 195
Other:
- board text added: "DMA/ROM control"
- board text added: "in"
- board text added: "out"
