File: RAM128.sch (KiCad schematic (older format))
At the start: 33 parts, among them J1 AppleIIBus, U1 621024, U10 74HCT32PW, U11 74AHCT1G126GW, U2 74HCT245PW, U3 74HCT273PW, U4 74HCT273PW, U5 74HCT04PW, U6 74HCT08PW, U7 74HCT32PW, U8 74HCT08PW, U9 74HCT08PW

Commit message: Good but ugly
Parts:
- removed U5: 74HCT04PW, stdpads:TSSOP-14_4.4x5mm_P0.65mm, symbol 74xx:74LS04
- removed unit 4 of U7
- added JP1: D, Jumper:SolderJumper-2_P1.3mm_Bridged_RoundedPad1.0x1.5mm, symbol Device:Jumper_NC_Small
- added JP2: D, Jumper:SolderJumper-2_P1.3mm_Open_RoundedPad1.0x1.5mm, symbol Device:Jumper_NO_Small
- added R2: 3k3, stdpads:R_0805, symbol Device:R_Small
- added U12, U13, U14, U15, U16, U17, U19, U20: 741G04GW, stdpads:SOT-353, symbol GW_Logic:741G04GW
- U1: footprint stdpads:TSOP-I-32_18.4x8mm_P0.5mm -> stdpads:SOP-32_P1.27mm; symbol GW_RAM:SRAM-128Kx8-TSOP1-32 -> GW_RAM:SRAM-128Kx8-SOP-32; LCSC Part C261864 -> C397875
- U10, U7: value 74HCT32PW -> 74AHCT32PW; LCSC Part C132266 -> C129435
- U2: LCSC Part C426701 -> C5980
- U6, U8, U9: value 74HCT08PW -> 74AHCT08PW; LCSC Part C8181 -> C155175
- U7: value 74HCT32PW -> 74AHCT32PW; LCSC Part C8181 -> C129435
Connections:
- net +5V: now also U1.30 (CS), U1.32 (VCC), U12.5 (Vcc), U13.5 (Vcc), U14.5 (Vcc), U15.5 (Vcc), U16.5 (Vcc), U17.5 (Vcc), U19.5 (Vcc), U20.5 (Vcc); no longer U1.6 (CS), U1.8 (VCC)
- net A0: now also U1.12 (A0), U4.7 (D2), U6.10, U13.2 (A); no longer U1.1 (A11), U4.3 (D0), U6.13
- net A1: now also U1.23 (A10), U14.2 (A); no longer U1.2 (A9)
- net A10: now also U1.28 (A13); no longer U1.19 (A1)
- net A11: now also U1.6 (A6); no longer U1.20 (A0)
- net A12: now also U8.1; no longer U8.5
- net A13: now also U8.2, U15.2 (A); no longer U8.4
- net A14: now also U8.13; no longer U8.12
- net A15: now also U8.12; no longer U8.13
- net A2: now also U1.11 (A1), U12.2 (A); no longer U1.3 (A8)
- net A3: now also U1.10 (A2), U4.3 (D0); no longer U1.4 (A13), U4.7 (D2)
- net A4: now also U1.25 (A11); no longer U1.16 (A4)
- net A5: now also U1.9 (A3); no longer U1.15 (A5)
- net A6: now also U1.26 (A9); no longer U1.13 (A7)
- net A7: now also U1.8 (A4); no longer U1.7 (A15)
- net A8: now also U1.27 (A8); no longer U1.17 (A3)
- net A9: now also U1.7 (A5); no longer U1.18 (A2)
- net BankAB: now also U8.5; no longer U8.2
- net DMAin: now also U9.5, U19.2 (A); no longer J1.24 (Pin_24), U6.10
- net ENWR1: now also U6.9; no longer U6.12
- net ENWR1A0: now also U6.8; no longer U6.11
- net GND: now also U1.16 (GND), R2.2, U12.3 (GND), U13.3 (GND), U14.3 (GND), U15.3 (GND), U16.3 (GND), U17.3 (GND), U19.3 (GND), U20.3 (GND); no longer U1.32 (~OE)
- net INHOE: now also U6.12, JP2.1; no longer U6.9
- net PHI0: now also U6.13; no longer U9.5
- net RA12: now also U1.5 (A7); no longer U1.14 (A6)
- net RA14: now also U1.4 (A12), U4.6 (Q2); no longer U1.12 (A12), U4.2 (Q0)
- net RA15: now also U1.3 (A14); no longer U1.11 (A14)
- net RA16: now also U1.2 (A16), U4.2 (Q0); no longer U1.10 (A16), U4.6 (Q2)
- net RD0: now also U1.13 (D0), U2.7 (A5); no longer U1.26 (D4), U2.5 (A3)
- net RD1: now also U1.14 (D1), U2.8 (A6); no longer U1.27 (D5), U2.4 (A2)
- net RD2: now also U1.15 (D2), U2.9 (A7); no longer U1.28 (D6), U2.3 (A1)
- net RD3: now also U1.17 (D3); no longer U1.29 (D7)
- net RD4: now also U1.18 (D4), U2.3 (A1); no longer U1.21 (D0), U2.9 (A7)
- net RD5: now also U1.19 (D5), U2.4 (A2); no longer U1.22 (D1), U2.8 (A6)
- net RD6: now also U1.20 (D6), U2.5 (A3); no longer U1.23 (D2), U2.7 (A5)
- net RD7: now also U1.21 (D7); no longer U1.25 (D3)
- net R~CS~: now also U1.22 (~CS~), U17.4 (Y); no longer U1.30 (~CS~)
- net R~W~: now also U1.29 (~WE), U16.2 (A); no longer U1.5 (~WE)
- net at U7.1: now also U12.4 (Y)
- net at U10.4: now also U8.6; no longer U8.3
- net at U10.5: now also U8.3; no longer U8.6
- net at U8.10: now also U16.4 (Y)
- net at U9.4: now also U6.11, JP1.1, JP2.2; no longer U6.8
- net at U6.1: now also U13.4 (Y)
- net at U6.2: now also U14.4 (Y)
- net at U7.10: now also U19.4 (Y)
- net at U7.8: now also U20.2 (A)
- net at U7.9: now also JP1.2, R2.1
- net RCS: no longer names the net of U9.6
- net RCS: now also U17.2 (A)
- new net: U15.4 (Y), U8.4
- new net DMAout: J1.24 (Pin_24), U20.4 (Y)
Other:
- moved on the sheet: R1, U10B, U10C, U10D, U11, U7A, U7C, U8C, U8D, U9A, U9B, U9C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
