File: RAM128.sch (KiCad schematic (older format))
At the start: 43 parts, among them J1 AppleIIBus, U1 621024, U10 74AHCT32PW, U11 74AHCT1G126GW, U12 741G04GW, U13 741G04GW, U14 741G04GW, U15 741G04GW, U16 741G04GW, U17 741G04GW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

Commit message: Fabbed
Parts:
- removed C1: 2u2, stdpads:C_0603, symbol Device:C_Small
- removed JP1: D, Jumper:SolderJumper-2_P1.3mm_Bridged_RoundedPad1.0x1.5mm, symbol Device:Jumper_NC_Small
- removed JP2: D, Jumper:SolderJumper-2_P1.3mm_Open_RoundedPad1.0x1.5mm, symbol Device:Jumper_NO_Small
- added C11, C12, C13, C14, C15, C5: 2u2, stdpads:C_0603, symbol Device:C_Small
- added R3, R4: 22k, stdpads:R_0805, symbol Device:R_Small
- added R5, R6, R7: 33, stdpads:R_0805, symbol Device:R_Small
- added unit 4 of U7
- H4: footprint stdpads:PasteHole_1.1mm_PTH -> stdpads:PasteHole_1.152mm_NPTH
- R2: value 3k3 -> 22k; LCSC Part C26010 -> C17560
- U11: value 74AHCT1G126GW -> 74LVC1G126GW; LCSC Part C7485 -> C88039
- U12, U13, U14, U15, U16, U17, U19, U20: value 741G04GW -> 74AHCT1G04GW
- renumbered C11 to C1, C12 to C16
Connections:
- net +5V: now also C11.1, C12.1, C13.1, C14.1, C15.1, C5.1, R3.1, R4.1
- net A13: now also U7.13
- net D0: now also U2.18 (B0); no longer U2.11 (B7)
- net D1: now also U2.17 (B1); no longer U2.12 (B6)
- net D2: now also U2.16 (B2); no longer U2.13 (B5)
- net D3: now also U2.15 (B3); no longer U2.14 (B4)
- net D4: now also U2.14 (B4); no longer U2.15 (B3)
- net D5: now also U2.13 (B5); no longer U2.16 (B2)
- net D6: now also U2.12 (B6); no longer U2.17 (B1)
- net D7: now also U2.11 (B7); no longer U2.18 (B0)
- net DMAin: now also R3.2, R6.2; no longer U9.5
- net GND: now also C11.2, C12.2, C13.2, C14.2, C15.2, C5.2
- net PHI0: now also U9.5; no longer U6.13
- net RD0: now also U2.6 (A4); no longer U2.7 (A5)
- net RD2: now also U2.3 (A1); no longer U2.9 (A7)
- net RD4: now also U2.4 (A2); no longer U2.3 (A1)
- net RD5: now also U2.9 (A7); no longer U2.4 (A2)
- net RD6: now also U2.7 (A5); no longer U2.5 (A3)
- net RD7: now also U2.5 (A3); no longer U2.6 (A4)
- net R~W~: now also U7.12
- net ~INH~: now also R5.1; no longer U11.4 (Y)
- net ~A2~: now reaches U12.4 (Y), U7.1
- net at R2.1, U7.9: now also R7.2
- net ~A13~: now reaches U15.4 (Y), U8.4
- net ~A0~: now reaches U13.4 (Y), U6.1
- net ~A1~: now reaches U14.4 (Y), U6.2
- net ~DMAout~: now reaches U20.2 (A), U7.8
- net ~R~W: now reaches U16.4 (Y), U8.10
- net RCS: now reaches U17.2 (A), U9.6
- net RCS: now also R7.1
- new net: R5.2, U11.4 (Y)
- new net: R4.2, R6.1, U6.13
- no-connect marks 9 -> 10
Other:
- moved on the sheet: C1, C10, C16, C2, C3, C4, C6, C7, C8, C9, FID1, FID2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

Commit message: Fabbed
Parts:
- removed R6, R7: 33, stdpads:R_0805, symbol Device:R_Small
- added SW1: DMA/ROM, stdpads:SW_DIP_SPSTx02_Slide_DSHP02TS_P1.27mm, symbol Switch:SW_DIP_x02
- R3: value 22k -> 10k; LCSC Part C17560 -> C17414
Connections:
- net DMAin: now also SW1.4
- net RCS: now also SW1.3
- net at R2.1, U7.9: now also SW1.2
- net at R4.2, U6.13: now also SW1.1
- no-connect marks 10 -> 11
Other:
- moved on the sheet: R3, R4
Changed lines of the file:
@@
 Sheet 1 1
 Title "RAM128 (GW4208B)"
-Date "2021-01-05"
+Date "2021-02-24"
 Rev "1.0"
 Comp "Garrett's Workshop"
@@
 Text Label 2850 3050 0    50   ~ 0
 RD7
-Text Label 4200 5500 2    50   ~ 0
+Text Label 3500 5500 0    50   ~ 0
 DMAin
 Text Label 5400 5600 2    50   ~ 0
@@
 Wire Wire Line
 	6700 6000 6700 6100
-Wire Wire Line
-	6000 5500 6050 5500
-Wire Wire Line
-	6050 5500 6700 5500
-Connection ~ 6050 5500
-$Comp
-L Device:R_Small R7
-U 1 1 60294FE3
-P 6050 5600
-F 0 "R7" H 6109 5646 50  0000 L CNN
-F 1 "33" H 6109 5555 50  0000 L CNN
-F 2 "stdpads:R_0805" H 6050 5600 50  0001 C CNN
-F 3 "~" H 6050 5600 50  0001 C CNN
-F 4 "C17634" H 6050 5600 50  0001 C CNN "LCSC Part"
-	1    6050 5600
-	1    0    0    -1
-$EndComp
 Text Label 4800 5300 2    50   ~ 0
 INHOE
-$Comp
-L Device:R_Small R6
-U 1 1 602CF046
-P 4350 5500
-F 0 "R6" V 4300 5500 50  0000 C BNN
-F 1 "33" V 4350 5500 40  0000 C CNN
-F 2 "stdpads:R_0805" H 4350 5500 50  0001 C CNN
-F 3 "~" H 4350 5500 50  0001 C CNN
-F 4 "C17634" H 4350 5500 50  0001 C CNN "LCSC Part"
-	1    4350 5500
-	0    1    -1   0
-$EndComp
-$Comp
-L Device:R_Small R3
-U 1 1 6035C673
-P 4200 5350
-F 0 "R3" H 4259 5396 50  0000 L CNN
-F 1 "22k" H 4259 5305 50  0000 L CNN
-F 2 "stdpads:R_0805" H 4200 5350 50  0001 C CNN
-F 3 "~" H 4200 5350 50  0001 C CNN
-F 4 "C17560" H 4200 5350 50  0001 C CNN "LCSC Part"
-	1    4200 5350
-	-1   0    0    -1
-$EndComp
-$Comp
-L power:+5V #PWR0135
-U 1 1 6035C679
-P 4200 5250
-F 0 "#PWR0135" H 4200 5100 50  0001 C CNN
-F 1 "+5V" H 4200 5400 50  0000 C CNN
-F 2 "" H 4200 5250 50  0001 C CNN
-F 3 "" H 4200 5250 50  0001 C CNN
-	1    4200 5250
-	1    0    0    -1
-$EndComp
-Wire Wire Line
-	4500 5450 4500 5500
-Wire Wire Line
-	4200 5450 4200 5500
-Wire Wire Line
-	4250 5500 4200 5500
 $Comp
 L 74xx:74LS08 U6
@@
 $EndComp
 $Comp
-L 74xx:74LS08 U9
-U 2 1 61AB3A41
-P 5700 5500
-F 0 "U9" H 5700 5500 50  0000 C CNN
-F 1 "74AHCT08PW" H 5700 5700 50  0000 C CNN
-F 2 "stdpads:TSSOP-14_4.4x5mm_P0.65mm" H 5700 5500 50  0001 C CNN
-F 3 "http://www.ti.com/lit/gpn/sn74LS08" H 5700 5500 50  0001 C CNN
-F 4 "C155175" H 5700 5500 50  0001 C CNN "LCSC Part"
-	2    5700 5500
-	1    0    0    -1
-$EndComp
-$Comp
-L Device:R_Small R4
-U 1 1 602BB8BD
-P 4500 5350
-F 0 "R4" H 4559 5396 50  0000 L CNN
-F 1 "22k" H 4559 5305 50  0000 L CNN
-F 2 "stdpads:R_0805" H 4500 5350 50  0001 C CNN
-F 3 "~" H 4500 5350 50  0001 C CNN
-F 4 "C17560" H 4500 5350 50  0001 C CNN "LCSC Part"
-	1    4500 5350
-	-1   0    0    -1
-$EndComp
-$Comp
 L power:GND #PWR0123
 U 1 1 5FB31C47
@@
 	1    0    0    -1
 $EndComp
-Wire Wire Line
-	4450 5500 4500 5500
 Wire Wire Line
 	6100 6100 6000 6100
@@
 Wire Wire Line
 	4500 5500 4800 5500
-Connection ~ 4500 5500
-Wire Wire Line
-	4500 5250 4200 5250
-Connection ~ 4200 5250
 $Comp
 L 74xx:74LS32 U10
@@
 Wire Wire Line
 	8150 1850 8200 1850
+$Comp
+L Switch:SW_DIP_x02 SW1
+U 1 1 6678EBA0
+P 4200 5600
+F 0 "SW1" H 4200 5850 50  0000 C CNN
+F 1 "DMA/ROM" H 4200 5450 50  0000 C CNN
+F 2 "stdpads:SW_DIP_SPSTx02_Slide_DSHP02TS_P1.27mm" H 4200 5600 50  0001 C CNN
+F 3 "~" H 4200 5600 50  0001 C CNN
+F 4 "C319052" H 4200 5600 50  0001 C CNN "LCSC Part"
+	1    4200 5600
+	-1   0    0    -1
+$EndComp
+Wire Wire Line
+	6000 5500 6700 5500
+$Comp
+L Device:R_Small R4
+U 1 1 602BB8BD
+P 4500 5400
+F 0 "R4" H 4559 5446 50  0000 L CNN
+F 1 "22k" H 4559 5355 50  0000 L CNN
+F 2 "stdpads:R_0805" H 4500 5400 50  0001 C CNN
+F 3 "~" H 4500 5400 50  0001 C CNN
+F 4 "C17560" H 4500 5400 50  0001 C CNN "LCSC Part"
+	1    4500 5400
+	1    0    0    -1
+$EndComp
+NoConn ~ 5250 5900
+Wire Wire Line
+	3500 5600 3900 5600
+Text Label 3500 5600 0    50   ~ 0
+RCS
+Connection ~ 4500 5500
+$Comp
+L 74xx:74LS08 U9
+U 2 1 61AB3A41
+P 5700 5500
+F 0 "U9" H 5700 5500 50  0000 C CNN
+F 1 "74AHCT08PW" H 5700 5700 50  0000 C CNN
+F 2 "stdpads:TSSOP-14_4.4x5mm_P0.65mm" H 5700 5500 50  0001 C CNN
+F 3 "http://www.ti.com/lit/gpn/sn74LS08" H 5700 5500 50  0001 C CNN
+F 4 "C155175" H 5700 5500 50  0001 C CNN "LCSC Part"
+	2    5700 5500
+	1    0    0    -1
+$EndComp
+Wire Wire Line
+	3800 6000 5200 6000
+Connection ~ 3800 5500
+Wire Wire Line
+	3800 5500 3900 5500
+Wire Wire Line
+	3500 5500 3800 5500
+Wire Wire Line
+	3800 5500 3800 6000
+$Comp
+L Device:R_Small R3
+U 1 1 6035C673
+P 3800 5400
+F 0 "R3" H 3859 5446 50  0000 L CNN
+F 1 "10k" H 3859 5355 50  0000 L CNN
+F 2 "stdpads:R_0805" H 3800 5400 50  0001 C CNN
+F 3 "~" H 3800 5400 50  0001 C CNN
+F 4 "C17414" H 3800 5400 50  0001 C CNN "LCSC Part"
+	1    3800 5400
+	1    0    0    -1
+$EndComp
+Wire Wire Line
+	4500 5300 3800 5300
+Connection ~ 3800 5300
+$Comp
+L power:+5V #PWR0135
+U 1 1 6035C679
+P 3800 5300
+F 0 "#PWR0135" H 3800 5150 50  0001 C CNN
+F 1 "+5V" H 3800 5450 50  0000 C CNN
+F 2 "" H 3800 5300 50  0001 C CNN
+F 3 "" H 3800 5300 50  0001 C CNN
+	1    3800 5300
+	1    0    0    -1
+$EndComp
+Wire Wire Line
+	4600 5600 4500 5600
+Wire Wire Line
+	6050 5700 4600 5700
+Wire Wire Line
+	4600 5700 4600 5600
+Wire Bus Line
+	650  3500 650  4450
 Wire Bus Line
 	3150 2650 3150 3350
@@
 	1850 2950 1850 4450
 Wire Bus Line
+	4550 2200 4550 4050
+Wire Bus Line
 	1750 2200 1750 4000
-Wire Bus Line
-	650  3500 650  4450
-Wire Bus Line
-	4550 2200 4550 4050
 $EndSCHEMATC
